File: melefant.kicad_pcb (KiCad board)
At the start: 2 copper layers, 156 x 109 mm, 46 parts, among them J1 AudioJack4, U1 Arduino_Pro_Micro

Commit message: pcb done.
Parts:
- added REF**: hole, utilities:hole, F.Cu at (104.5, -43.2)
- added REF**: hole, utilities:hole, F.Cu at (-13.0, -45.5)
- added REF**: hole, utilities:hole, F.Cu at (-13.0, -86.0)
- added REF**: hole, utilities:hole, F.Cu at (25.0, -76.0)
- added REF**: hole, utilities:hole, F.Cu at (39.0, -86.0)
- added REF**: hole, utilities:hole, F.Cu at (95.5, -86.0)
- added REF**: hole, utilities:hole, F.Cu at (123.0, -63.0)
- added REF**: hole, utilities:hole, F.Cu at (128.5, -7.00)
- added REF**: hole, utilities:hole, F.Cu at (38.0, 5.00)
- added REF**: hole, utilities:hole, F.Cu at (6.00, 5.00)
- added REF**: hole, utilities:hole, F.Cu at (85.5, -43.2)
- added REF**: hole, utilities:hole, F.Cu at (66.5, -43.2)
- added REF**: hole, utilities:hole, F.Cu at (47.5, -46.3)
- added REF**: hole, utilities:hole, F.Cu at (28.5, -41.0)
- added REF**: hole, utilities:hole, F.Cu at (9.50, -23.7)
- added REF**: hole, utilities:hole, F.Cu at (104.0, 12.0)
- added REF**: hole, utilities:hole, F.Cu at (141.5, 15.0)
- added REF**: hole, utilities:hole, F.Cu at (-13.0, -9.50)
- moved D2 6.94 mm to (110.2, -15.6), turned to 270 degrees
- moved D1 5.55 mm to (22.8, -83.5), turned to 0 degrees
- moved U1 4.50 mm to (-1.05, -72.4)
- moved SW_RES1 4.41 mm to (19.5, -64.2), turned to 180 degrees
- moved LS1 4.17 mm to (22.7, -65.6)
- moved J1 3.27 mm to (115.0, -70.1)
- moved R4 2.15 mm to (22.8, -61.0)
Routing:
- net LEDB: track 42.1 -> 26.3 mm, vias 0 -> 1
- net LEDG(rotB): track 106.4 -> 93.7 mm, vias 0 -> 1
- net SWOUT: track 128.9 -> 140.6 mm
- net RST: track 18.0 -> 25.9 mm
- net row2: track 130.0 -> 136.8 mm
- net row3: track 128.1 -> 134.8 mm
- net Net-(D1-Pad1): track 9.87 -> 3.29 mm
- net row1: track 111.5 -> 118.0 mm
- net LEDR(rotA): track 101.7 -> 95.3 mm
- net row5: track 171.8 -> 176.3 mm
- net col1: track 38.9 -> 43.4 mm
- net Net-(D1-Pad4): track 11.9 -> 15.6 mm
- net col6: track 212.7 -> 216.2 mm
- net col5: track 189.7 -> 193.2 mm
- net col4: track 168.0 -> 171.5 mm
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Other:
- board size 156 x 109 mm -> 164 x 112.5 mm

Commit message: top plate
Parts:
- removed the REF** at (25.0, -76.0)
- moved REF** 144.7 mm to (186.2, 131.1)
- moved SD5:4 144.2 mm to (155.3, 129.6)
- moved SD5:7 144.2 mm to (211.8, 128.8)
- moved D1 144.2 mm to (102.8, 36.5)
- moved LS1 144.2 mm to (102.7, 54.4)
- moved R1 144.2 mm to (93.0, 46.7)
- moved R2 144.2 mm to (96.3, 46.7)
- moved R3 144.2 mm to (99.5, 46.8)
- moved R4 144.2 mm to (102.8, 59.0)
- moved R5 144.2 mm to (169.9, 41.8)
- moved R6 144.2 mm to (180.0, 38.8)
- moved REF** 144.2 mm to (184.5, 76.8)
- moved REF** 144.2 mm to (67.0, 74.5)
- moved REF** 144.2 mm to (67.0, 34.0)
- moved REF** 144.2 mm to (119.0, 34.0)
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Routing:
- net SDA: track 135.8 -> 138.6 mm
- net SCL: track 137.7 -> 140.5 mm
- net SWIN: track 250.8 -> 251.7 mm
Other:
- board size 164 x 112.5 mm -> 164.5 x 113 mm
